Commit message: Clean commits

File: iiwa_description/urdf/iiwa7.urdf.xacro (robot description, xacro)
@@ -39,5 +39,5 @@
   <link name="world"/>
   <!--iiwa-->
-  <xacro:iiwa7 hardware_interface="$(arg hardware_interface)" robot_name="$(arg robot_name)" parent="world" collision_postfix="$(arg collision_postfix)">
+  <xacro:iiwa7 hardware_interface="$(arg hardware_interface)" robot_name="$(arg robot_name)" parent="world">
     <origin xyz="$(arg origin_xyz)" rpy="$(arg origin_rpy)" />
   </xacro:iiwa7>

File: iiwa_description/urdf/iiwa7.xacro (robot description, xacro)
@@ -57,5 +57,5 @@
   <xacro:property name="max_velocity_6" value="${PI}"/>
   <xacro:property name="max_velocity_7" value="${PI}"/>
-  <xacro:macro name="iiwa7" params="parent hardware_interface robot_name collision_postfix *origin">
+  <xacro:macro name="iiwa7" params="parent hardware_interface robot_name *origin">
     <!--joint between {parent} and link_0-->
     <joint name="${parent}_${robot_name}_joint" type="fixed">
